File: airflowSensor.kicad_sch (KiCad schematic)
At the start: 5 parts, among them IC1 FS3000-1015

Commit message: fixed errors
Parts:
- renumbered IC1 to IC2
Connections:
- no-connect marks 2 -> 4
Changed lines of the file:
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@@
   )
   (no_connect (at 132.08 97.79))
+  (no_connect (at 160.02 97.79))
   (no_connect (at 132.08 95.25))
+  (no_connect (at 160.02 100.33))
   (wire (pts (xy 185.42 92.71) (xy 185.42 95.25))
     (stroke (width 0) (type default))
@@
   (symbol (lib_id "utsvt-chips:FS3000-1015") (at 132.08 87.63 0) (unit 1)
     (in_bom yes) (on_board yes) (dnp no) (fields_autoplaced)
-    (property "Reference" "IC1" (at 146.05 80.01 0)
+    (property "Reference" "IC2" (at 146.05 80.01 0)
       (effects (font (size 1.27 1.27)))
     )
@@
       (project "Telemetry-Peripheral-SOM-Daughterboard-IMU"
         (path "/637f68f0-cb9c-412a-8573-5d8e7ef6d8a2/9b10eeac-b1da-4b4a-b651-04148a20ecbc"
-          (reference "IC1") (unit 1)
+          (reference "IC2") (unit 1)
         )
       )

Commit message: assigned footprints for all capacitors
Parts:
- C5, C6: footprint (none) -> Capacitor_SMD:C_0805_2012Metric
Changed lines of the file:
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@@
       (effects (font (size 1.27 1.27)) (justify left))
     )
-    (property "Footprint" "" (at 191.4652 95.25 0)
+    (property "Footprint" "Capacitor_SMD:C_0805_2012Metric" (at 191.4652 95.25 0)
       (effects (font (size 1.27 1.27)) hide)
     )
@@
       (effects (font (size 1.27 1.27)) (justify left))
     )
-    (property "Footprint" "" (at 166.0652 113.03 0)
+    (property "Footprint" "Capacitor_SMD:C_0805_2012Metric" (at 166.0652 113.03 0)
       (effects (font (size 1.27 1.27)) hide)
     )

Commit message: first draft
Parts:
- renumbered IC2 to IC1
Changed lines of the file:
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@@
   (symbol (lib_id "utsvt-chips:FS3000-1015") (at 132.08 87.63 0) (unit 1)
     (in_bom yes) (on_board yes) (dnp no) (fields_autoplaced)
-    (property "Reference" "IC2" (at 146.05 80.01 0)
+    (property "Reference" "IC1" (at 146.05 80.01 0)
       (effects (font (size 1.27 1.27)))
     )
@@
       (project "Telemetry-Peripheral-SOM-Daughterboard-IMU"
         (path "/637f68f0-cb9c-412a-8573-5d8e7ef6d8a2/9b10eeac-b1da-4b4a-b651-04148a20ecbc"
-          (reference "IC2") (unit 1)
+          (reference "IC1") (unit 1)
         )
       )

Commit message: a
Parts:
- added TP1: TestPoint, TestPoint:TestPoint_Pad_2.0x2.0mm, symbol Connector:TestPoint
Connections:
- net +3.3V: now also TP1.1
Changed lines of the file:
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@@
 (kicad_sch (version 20230121) (generator eeschema)
   (paper "A4")
+  (junction (at 85.09 85.09) (diameter 0) (color 0 0 0 0)
+  )
   (junction (at 85.09 100.33) (diameter 0) (color 0 0 0 0)
   )
@@
     (stroke (width 0) (type default))
   )
+  (wire (pts (xy 85.09 85.09) (xy 85.09 90.17))
+    (stroke (width 0) (type default))
+  )
   (wire (pts (xy 185.42 90.17) (xy 185.42 87.63))
     (stroke (width 0) (type default))
@@
     (stroke (width 0) (type default))
   )
-  (wire (pts (xy 85.09 81.28) (xy 85.09 90.17))
+  (wire (pts (xy 85.09 81.28) (xy 85.09 85.09))
     (stroke (width 0) (type default))
   )
@@
         )
       )
+    )
+  )
+  (symbol (lib_id "Connector:TestPoint") (at 85.09 85.09 90) (unit 1)
+    (in_bom yes) (on_board yes) (dnp no) (fields_autoplaced)
+    (property "Reference" "TP1" (at 81.788 80.01 90)
+      (effects (font (size 1.27 1.27)))
+    )
+    (property "Value" "TestPoint" (at 81.788 82.55 90)
+      (effects (font (size 1.27 1.27)))
+    )
+    (property "Footprint" "TestPoint:TestPoint_Pad_2.0x2.0mm" (at 85.09 80.01 0)
+      (effects (font (size 1.27 1.27)) hide)
+    )
+    (property "Datasheet" "~" (at 85.09 80.01 0)
+      (effects (font (size 1.27 1.27)) hide)
+    )
+    (pin "1")
+    (instances
+      (project "Telemetry-Peripheral-SOM-Daughterboard-IMU"
+        (path "/637f68f0-cb9c-412a-8573-5d8e7ef6d8a2/9b10eeac-b1da-4b4a-b651-04148a20ecbc"
+          (reference "TP1") (unit 1)
+        )
+      )
