File: airflowSensor.kicad_sch (KiCad schematic)
At the start: 5 parts, among them IC1 FS3000-1015

Commit message: revision
Parts:
- added TP4, TP5: TestPoint, TestPoint:TestPoint_THTPad_D2.0mm_Drill1.0mm, symbol Connector:TestPoint
Connections:
- net airflowSensor_SCL: now also TP5.1
- net airflowSensor_SDA: now also TP4.1
Changed lines of the file:
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@@
 (kicad_sch (version 20230121) (generator eeschema)
   (paper "A4")
+  (junction (at 161.29 87.63) (diameter 0) (color 0 0 0 0)
+  )
+  (junction (at 130.81 100.33) (diameter 0) (color 0 0 0 0)
+  )
   (junction (at 85.09 100.33) (diameter 0) (color 0 0 0 0)
   )
@@
   (no_connect (at 132.08 95.25))
   (no_connect (at 160.02 100.33))
+  (wire (pts (xy 166.37 87.63) (xy 161.29 87.63))
+    (stroke (width 0) (type default))
+  )
   (wire (pts (xy 185.42 92.71) (xy 185.42 95.25))
     (stroke (width 0) (type default))
   )
+  (wire (pts (xy 127 100.33) (xy 130.81 100.33))
+    (stroke (width 0) (type default))
+  )
   (wire (pts (xy 95.25 87.63) (xy 132.08 87.63))
     (stroke (width 0) (type default))
@@
     (stroke (width 0) (type default))
   )
+  (wire (pts (xy 130.81 100.33) (xy 132.08 100.33))
+    (stroke (width 0) (type default))
+  )
   (wire (pts (xy 85.09 90.17) (xy 132.08 90.17))
     (stroke (width 0) (type default))
   )
   (wire (pts (xy 160.02 92.71) (xy 185.42 92.71))
+    (stroke (width 0) (type default))
+  )
+  (wire (pts (xy 161.29 87.63) (xy 160.02 87.63))
     (stroke (width 0) (type default))
   )
@@
     (effects (font (size 5 5) (thickness 1) bold) (justify left bottom))
   )
-  (hierarchical_label "airflowSensor_SDA" (shape output) (at 132.08 100.33 180) (fields_autoplaced)
+  (hierarchical_label "airflowSensor_SDA" (shape output) (at 127 100.33 180) (fields_autoplaced)
     (effects (font (size 1.27 1.27)) (justify right))
   )
-  (hierarchical_label "airflowSensor_SCL" (shape output) (at 160.02 87.63 0) (fields_autoplaced)
+  (hierarchical_label "airflowSensor_SCL" (shape output) (at 166.37 87.63 0) (fields_autoplaced)
     (effects (font (size 1.27 1.27)) (justify left))
   )
@@
     )
   )
+  (symbol (lib_id "Connector:TestPoint") (at 130.81 100.33 180) (unit 1)
+    (in_bom yes) (on_board yes) (dnp no) (fields_autoplaced)
+    (property "Reference" "TP4" (at 133.35 102.362 0)
+      (effects (font (size 1.27 1.27)) (justify right))
+    )
+    (property "Value" "TestPoint" (at 133.35 104.902 0)
+      (effects (font (size 1.27 1.27)) (justify right))
+    )
+    (property "Footprint" "TestPoint:TestPoint_THTPad_D2.0mm_Drill1.0mm" (at 125.73 100.33 0)
+      (effects (font (size 1.27 1.27)) hide)
+    )
+    (property "Datasheet" "~" (at 125.73 100.33 0)
+      (effects (font (size 1.27 1.27)) hide)
+    )
+    (pin "1")
+    (instances
+      (project "Telemetry-Peripheral-SOM-Daughterboard-IMU"
+        (path "/637f68f0-cb9c-412a-8573-5d8e7ef6d8a2/9b10eeac-b1da-4b4a-b651-04148a20ecbc"
+          (reference "TP4") (unit 1)
+        )
+      )
+    )
+  )
   (symbol (lib_id "Device:C_Small") (at 85.09 95.25 0) (unit 1)
     (in_bom yes) (on_board yes) (dnp no)
@@
         )
       )
+    )
+  )
+  (symbol (lib_id "Connector:TestPoint") (at 161.29 87.63 0) (unit 1)
+    (in_bom yes) (on_board yes) (dnp no) (fields_autoplaced)
+    (property "Reference" "TP5" (at 163.83 83.058 0)
+      (effects (font (size 1.27 1.27)) (justify left))
+    )
+    (property "Value" "TestPoint" (at 163.83 85.598 0)
+      (effects (font (size 1.27 1.27)) (justify left))
+    )
+    (property "Footprint" "TestPoint:TestPoint_THTPad_D2.0mm_Drill1.0mm" (at 166.37 87.63 0)
+      (effects (font (size 1.27 1.27)) hide)
+    )
+    (property "Datasheet" "~" (at 166.37 87.63 0)
+      (effects (font (size 1.27 1.27)) hide)
+    )
+    (pin "1")
+    (instances
+      (project "Telemetry-Peripheral-SOM-Daughterboard-IMU"
+        (path "/637f68f0-cb9c-412a-8573-5d8e7ef6d8a2/9b10eeac-b1da-4b4a-b651-04148a20ecbc"
+          (reference "TP5") (unit 1)
+        )
+      )

Commit message: added protective circuitry for temp sensors, made name changes for IMU
Parts:
- IC1: P/N (none) -> FS3000-1015
Changed lines of the file:
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@@
       (effects (font (size 1.27 1.27)) (justify left top) hide)
+    )
+    (property "P/N" "FS3000-1015" (at 132.08 87.63 0)
+      (effects (font (size 1.27 1.27)) hide)
     )
     (pin "1")
