File: Telemetry-Peripheral-SOM-Daughterboard-IMU.kicad_sch (KiCad schematic)
At the start: 5 parts, among them J1 Conn_02x10_Odd_Even

Commit message: Name changes
Other:
- sheet imuSensor ports: added IMU_MISO, IMU_MOSI, IMU_SCK; removed IMU_SCL, IMU_SDA, IMU_SDO/SA0
- note added: "V1.4 - Completed schematic (10/21/23)"
- note removed: "V1.4 -"
Changed lines of the file:
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@@
     (effects (font (size 1.27 1.27)) (justify left bottom))
   )
-  (text "V1.4 - " (at 179.07 83.82 0)
+  (text "V1.4 - Completed schematic (10/21/23)" (at 179.07 83.82 0)
     (effects (font (size 1.27 1.27)) (justify left bottom))
   )
@@
       (effects (font (size 1.27 1.27)) (justify left top))
     )
-    (pin "IMU_SDO{slash}SA0" output (at 127 77.47 180)
+    (pin "IMU_INT2" output (at 127 92.71 180)
+      (effects (font (size 1.27 1.27)) (justify left))
+    )
+    (pin "IMU_MOSI" input (at 127 96.52 180)
+      (effects (font (size 1.27 1.27)) (justify left))
+    )
+    (pin "IMU_CS" input (at 127 85.09 180)
+      (effects (font (size 1.27 1.27)) (justify left))
+    )
+    (pin "IMU_SCK" input (at 127 88.9 180)
       (effects (font (size 1.27 1.27)) (justify left))
     )
@@
       (effects (font (size 1.27 1.27)) (justify left))
     )
-    (pin "IMU_SCL" input (at 127 96.52 180)
-      (effects (font (size 1.27 1.27)) (justify left))
-    )
-    (pin "IMU_CS" input (at 127 85.09 180)
-      (effects (font (size 1.27 1.27)) (justify left))
-    )
-    (pin "IMU_INT2" output (at 127 92.71 180)
-      (effects (font (size 1.27 1.27)) (justify left))
-    )
-    (pin "IMU_SDA" input (at 127 88.9 180)
-      (effects (font (size 1.27 1.27)) (justify left))
-    )
+    (pin "IMU_MISO" output (at 127 77.47 180)
+      (effects (font (size 1.27 1.27)) (justify left))
+    )

Commit message: changes to I2C
Changed lines of the file:
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@@
     (effects (font (size 1.27 1.27)) (justify right bottom))
   )
-  (label "I2C1_SCL" (at 105.41 92.71 0) (fields_autoplaced)
+  (label "I2C1_SCL" (at 105.41 128.27 0) (fields_autoplaced)
     (effects (font (size 1.27 1.27)) (justify left bottom))
   )
-  (label "I2C1_SDA" (at 105.41 81.28 0) (fields_autoplaced)
+  (label "I2C1_SDA" (at 105.41 133.35 0) (fields_autoplaced)
     (effects (font (size 1.27 1.27)) (justify left bottom))
   )
@@
     (effects (font (size 1.27 1.27)) (justify left bottom))
   )
-  (label "I2C2_SDA" (at 105.41 133.35 0) (fields_autoplaced)
+  (label "I2C2_SDA" (at 105.41 81.28 0) (fields_autoplaced)
     (effects (font (size 1.27 1.27)) (justify left bottom))
   )
-  (label "I2C2_SCL" (at 105.41 128.27 0) (fields_autoplaced)
+  (label "I2C2_SCL" (at 105.41 92.71 0) (fields_autoplaced)
     (effects (font (size 1.27 1.27)) (justify left bottom))
   )
